File: Hot_Wheels_Electronics/Hot_Wheels_Electronics.kicad_sch (KiCad schematic)
At the start: 15 parts, among them J1 motor_output, M1 motor_driver: DRV8833PW, SW1 main_switch, U1 esp32-wemos-d1-mini, U3 BMI160, U4 QITN BEC

Commit message: added spi support to bmi160 imu
Connections:
- net +3V3: no longer U3.12 (CSB)
- net GND: no longer U3.1 (SDO), U3.6 (GNDIO)
- net i2c_scl: no longer U3.13 (SCx)
- net i2c_sda: no longer U3.14 (SDx)
- net imu_miso: now reaches U1.10 (IO_19/D6)
- net imu_miso: now also U3.1 (SDO)
- net imu_mosi: now reaches U1.12 (IO_23/D7)
- net imu_mosi: now also U3.14 (SDx)
- net imu_cs: now reaches U1.29 (IO_17/D3)
- net imu_cs: now also U3.12 (CSB)
- net imu_sck: now reaches U1.8 (IO_18/D5)
- net imu_sck: now also U3.13 (SCx)
Changed lines of the file:
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@@
-	)
-	(junction
-		(at 233.68 49.53)
-		(diameter 0)
-		(color 0 0 0 0)
 	)
 	(junction
@@
 	)
 	(junction
-		(at 234.95 72.39)
-		(diameter 0)
-		(color 0 0 0 0)
-	)
-	(junction
 		(at 87.63 149.86)
 		(diameter 0)
@@
 	)
 	(junction
-		(at 233.68 72.39)
-		(diameter 0)
-		(color 0 0 0 0)
-	)
-	(junction
 		(at 168.91 41.91)
 		(diameter 0)
@@
 	(wire
 		(pts
+			(xy 210.82 59.69) (xy 223.52 59.69)
+		)
+		(stroke
+			(width 0)
+			(type default)
+		)
+	)
+	(wire
+		(pts
+			(xy 115.57 85.09) (xy 135.89 85.09)
+		)
+		(stroke
+			(width 0)
+			(type default)
+		)
+	)
+	(wire
+		(pts
 			(xy 57.15 81.28) (xy 64.77 81.28)
 		)
@@
 	(wire
 		(pts
-			(xy 234.95 72.39) (xy 234.95 76.2)
-		)
-		(stroke
-			(width 0)
-			(type default)
-		)
-	)
-	(wire
-		(pts
 			(xy 55.88 142.24) (xy 55.88 144.78)
 		)
@@
 	(wire
 		(pts
+			(xy 115.57 62.23) (xy 135.89 62.23)
+		)
+		(stroke
+			(width 0)
+			(type default)
+		)
+	)
+	(wire
+		(pts
 			(xy 44.45 157.48) (xy 53.34 157.48)
 		)
@@
 	(wire
 		(pts
-			(xy 223.52 62.23) (xy 214.63 62.23)
+			(xy 223.52 62.23) (xy 210.82 62.23)
 		)
 		(stroke
@@
 	(wire
 		(pts
-			(xy 223.52 54.61) (xy 217.17 54.61)
-		)
-		(stroke
-			(width 0)
-			(type default)
-		)
-	)
-	(wire
-		(pts
 			(xy 162.56 36.83) (xy 167.64 36.83)
 		)
@@
 	(wire
 		(pts
-			(xy 205.74 57.15) (xy 223.52 57.15)
-		)
-		(stroke
-			(width 0)
-			(type default)
-		)
-	)
-	(wire
-		(pts
-			(xy 217.17 72.39) (xy 233.68 72.39)
+			(xy 115.57 59.69) (xy 135.89 59.69)
 		)
 		(stroke
@@
 	(wire
 		(pts
-			(xy 205.74 59.69) (xy 223.52 59.69)
+			(xy 210.82 57.15) (xy 223.52 57.15)
 		)
 		(stroke
@@
 	(wire
 		(pts
+			(xy 210.82 54.61) (xy 223.52 54.61)
+		)
+		(stroke
+			(width 0)
+			(type default)
+		)
+	)
+	(wire
+		(pts
 			(xy 55.88 149.86) (xy 58.42 149.86)
 		)
@@
 	(wire
 		(pts
-			(xy 214.63 62.23) (xy 214.63 49.53)
-		)
-		(stroke
-			(width 0)
-			(type default)
-		)
-	)
-	(wire
-		(pts
 			(xy 66.04 34.29) (xy 66.04 44.45)
 		)
@@
 	(wire
 		(pts
-			(xy 115.57 85.09) (xy 135.89 85.09)
-		)
-		(stroke
-			(width 0)
-			(type default)
-		)
-	)
-	(wire
-		(pts
 			(xy 168.91 41.91) (xy 162.56 41.91)
 		)
@@
 	(wire
 		(pts
-			(xy 217.17 54.61) (xy 217.17 72.39)
-		)
-		(stroke
-			(width 0)
-			(type default)
-		)
-	)
-	(wire
-		(pts
 			(xy 234.95 49.53) (xy 236.22 49.53)
 		)
@@
 	(wire
 		(pts
-			(xy 233.68 72.39) (xy 234.95 72.39)
-		)
-		(stroke
-			(width 0)
-			(type default)
-		)
-	)
-	(wire
-		(pts
 			(xy 78.74 115.57) (xy 78.74 128.27)
 		)
@@
 	(wire
 		(pts
-			(xy 234.95 72.39) (xy 236.22 72.39)
-		)
-		(stroke
-			(width 0)
-			(type default)
-		)
-	)
-	(wire
-		(pts
 			(xy 55.88 154.94) (xy 55.88 149.86)
 		)
@@
 	(wire
 		(pts
-			(xy 214.63 49.53) (xy 233.68 49.53)
+			(xy 115.57 87.63) (xy 135.89 87.63)
 		)
 		(stroke
@@
 	(wire
 		(pts
+			(xy 115.57 64.77) (xy 135.89 64.77)
+		)
+		(stroke
+			(width 0)
+			(type default)
+		)
+	)
+	(wire
+		(pts
 			(xy 53.34 139.7) (xy 58.42 139.7)
 		)
@@
 		)
 	)
-	(label "i2c_scl"
-		(at 205.74 59.69 0)
-		(effects
-			(font
-				(size 1.27 1.27)
-			)
-			(justify left bottom)
-		)
-	)
-	(label "i2c_sda"
-		(at 205.74 57.15 0)
+	(label "imu_miso"
+		(at 115.57 64.77 0)
 		(effects
 			(font
@@
 		)
 	)
+	(label "imu_cs"
+		(at 210.82 62.23 0)
+		(effects
+			(font
+				(size 1.27 1.27)
+			)
+			(justify left bottom)
+		)
+	)
+	(label "imu_sck"
+		(at 210.82 59.69 0)
+		(effects
+			(font
+				(size 1.27 1.27)
+			)
+			(justify left bottom)
+		)
+	)
 	(label "drv_curr"
 		(at 115.57 72.39 0)
@@
 		)
 	)
+	(label "imu_sck"
+		(at 115.57 62.23 0)
+		(effects
+			(font
+				(size 1.27 1.27)
+			)
+			(justify left bottom)
+		)
+	)
+	(label "imu_mosi"
+		(at 210.82 57.15 0)
+		(effects
+			(font
+				(size 1.27 1.27)
+			)
+			(justify left bottom)
+		)
+	)
 	(label "servo_signal"
 		(at 115.57 57.15 0)
@@
 		)
 	)
+	(label "imu_miso"
+		(at 210.82 54.61 0)
+		(effects
+			(font
+				(size 1.27 1.27)
+			)
+			(justify left bottom)
+		)
+	)
 	(label "drv_2"
 		(at 115.57 69.85 0)
@@
 		)
 	)
-	(label "i2c_scl"
-		(at 115.57 85.09 0)
+	(label "imu_cs"
+		(at 115.57 59.69 0)
 		(effects
 			(font
@@
 		)
 	)
+	(label "imu_mosi"
+		(at 115.57 87.63 0)
+		(effects
+			(font
+				(size 1.27 1.27)
+			)
+			(justify left bottom)
+		)
+	)
 	(label "drv_curr"
 		(at 22.86 147.32 0)
+		(effects
+			(font
+				(size 1.27 1.27)
+			)
+			(justify left bottom)
+		)
+	)
+	(label "i2c_scl"
+		(at 115.57 85.09 0)
 		(effects
 			(font
@@
 	(symbol
 		(lib_id "power:GND")
-		(at 234.95 76.2 0)
+		(at 236.22 72.39 0)
 		(unit 1)
 		(body_style 1)
@@
 		(fields_autoplaced yes)
 		(property "Reference" "#PWR019"
-			(at 234.95 82.55 0)
+			(at 236.22 78.74 0)
 			(hide yes)
 			(show_name no)
@@
 		)
 		(property "Value" "GND"
-			(at 234.95 81.28 0)
+			(at 236.22 77.47 0)
 			(show_name no)
 			(do_not_autoplace no)
@@
 		)
 		(property "Footprint" ""
-			(at 234.95 76.2 0)
+			(at 236.22 72.39 0)
 			(hide yes)
 			(show_name no)
@@
 		)
 		(property "Datasheet" ""
-			(at 234.95 76.2 0)
+			(at 236.22 72.39 0)
 			(hide yes)
 			(show_name no)
@@
 		)
 		(property "Description" "Power symbol creates a global label with name \"GND\" , ground"
-			(at 234.95 76.2 0)
-			(hide yes)
-			(show_name no)
+			(at 236.22 72.39 0)
+			(hide yes)
+			(show_name no)
